File: Hardware/Input Pinouts/Input Pinouts.kicad_sch (KiCad schematic)
At the start: 2 parts, among them J1 Relays, J2 Accessory

Commit message: Update
Changed lines of the file:
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@@
     (pin "9")
+  )
+  (symbol (lib_id "A.C. Wright Logo:LOGO") (at 278.13 173.99 0) (unit 1)
+    (in_bom yes) (on_board yes) (fields_autoplaced)
+    (property "Reference" "#G?" (id 0) (at 278.13 178.2318 0)
+      (effects (font (size 1.524 1.524)) hide)
+    )
+    (property "Value" "LOGO" (id 1) (at 278.13 169.7482 0)
+      (effects (font (size 1.524 1.524)) hide)
+    )
+    (property "Footprint" "A.C. Wright Logo:A.C. Wright Logo 10mm" (id 2) (at 278.13 173.99 0)
+      (effects (font (size 1.27 1.27)) hide)
+    )
+    (property "Datasheet" "" (id 3) (at 278.13 173.99 0)
+      (effects (font (size 1.27 1.27)) hide)
+    )
   )
   (symbol (lib_id "power:GND") (at 173.99 57.15 0) (unit 1)
@@
     )
     (pin "1")
+  )
+  (symbol (lib_id "Graphic:Logo_Open_Hardware_Small") (at 265.43 173.99 0) (unit 1)
+    (in_bom yes) (on_board yes) (fields_autoplaced)
+    (property "Reference" "#LOGO?" (id 0) (at 265.43 167.005 0)
+      (effects (font (size 1.27 1.27)) hide)
+    )
+    (property "Value" "Logo_Open_Hardware_Small" (id 1) (at 265.43 179.705 0)
+      (effects (font (size 1.27 1.27)) hide)
+    )
+    (property "Footprint" "Symbol:OSHW-Logo2_9.8x8mm_SilkScreen" (id 2) (at 265.43 173.99 0)
+      (effects (font (size 1.27 1.27)) hide)
+    )
+    (property "Datasheet" "~" (id 3) (at 265.43 173.99 0)
+      (effects (font (size 1.27 1.27)) hide)
+    )
   )
   (symbol (lib_id "power:GND") (at 113.03 57.15 0) (unit 1)
@@
   )
   (symbol_instances
+    (path "/86333961-c0bb-402d-988e-cb4b2d5e18ba"
+      (reference "#G?") (unit 1) (value "LOGO") (footprint "A.C. Wright Logo:A.C. Wright Logo 10mm")
+    )
+    (path "/b7a02604-4c24-4391-8423-093b770ba344"
+      (reference "#LOGO?") (unit 1) (value "Logo_Open_Hardware_Small") (footprint "Symbol:OSHW-Logo2_9.8x8mm_SilkScreen")
+    )
     (path "/cac89a66-b0ed-4c53-b214-3228113b78ce"
       (reference "#PWR01") (unit 1) (value "GND") (footprint "")

Commit message: Rev A boards ordered
Other:
- title: Input Pinouts -> Sherline CNC - Input Pinouts
Changed lines of the file:
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@@
   (paper "A4")
   (title_block
-    (title "Input Pinouts")
+    (title "Sherline CNC - Input Pinouts")
     (date "2021-12-03")
     (rev "A")
