File: Hardware/Input Board/Input Board.kicad_pcb (KiCad board)
At the start: 2 copper layers, 190 x 100 mm, 41 parts, among them J1 Relays, J10 Flood, J11 Other, J12 Encoder Input, J13 Signals, J14 Encoder Output, J15 X Limit, J16 Y Limit, J17 Z Limit, J18 Probe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

Commit message: Input board complete
Parts:
- J12: value Encoder Input -> Encoder
- J14: value Encoder Output -> Encoder
- moved G*** 206.6 mm to (58.0, 122.5)
- moved H4 193.1 mm to (224.0, 56.0)
- moved REF** 158.7 mm to (119.5, 122.5)
- moved J5 137.1 mm to (70.5, 80.3)
- moved J1 120.2 mm to (169.5, 68.5), turned to 180 degrees
- moved J7 108.2 mm to (70.5, 106.3)
- moved K2 107.2 mm to (86.0, 97.0)
- moved J11 92.6 mm to (64.0, 107.0), turned to 0 degrees
- moved H5 84.5 mm to (149.0, 118.0)
- moved J6 71.8 mm to (70.5, 93.3)
- moved J10 69.1 mm to (64.0, 94.0), turned to 0 degrees
- moved J9 45.6 mm to (64.0, 81.0), turned to 0 degrees
- moved J2 33.5 mm to (91.0, 55.5), turned to 180 degrees
- moved J4 31.1 mm to (70.5, 67.3)
- moved J17 23.1 mm to (223.5, 76.0)
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Routing:
- net 24V: track 0.00 -> 221.4 mm
- net 5V: track 0.00 -> 189.8 mm, vias 0 -> 1
- net Net-(J1-Pad20): track 0.00 -> 119.8 mm, vias 0 -> 2
- net FWD: track 0.00 -> 112.5 mm
- net Net-(J7-Pad2): track 0.00 -> 111.1 mm
- net Net-(J1-Pad6): track 0.00 -> 108.5 mm
- net Net-(J11-Pad1): track 0.00 -> 108.1 mm
- net FWD_REV_COM: track 0.00 -> 92.6 mm
- net Net-(J1-Pad9): track 0.00 -> 90.5 mm
- net Net-(J10-Pad1): track 0.00 -> 88.5 mm
- net Net-(J6-Pad2): track 0.00 -> 86.0 mm
- net REV: track 0.00 -> 76.0 mm, vias 0 -> 1
- net /ACC_GND: track 0.00 -> 75.7 mm, vias 0 -> 1
- net Net-(J1-Pad23): track 0.00 -> 72.3 mm
- net /ACC_24V: track 0.00 -> 53.8 mm
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- added copper zone on B.Cu, net GND
- added copper zone on F.Cu, net GND
Other:
- board size 190 x 100 mm -> 180 x 100 mm
- board text added: "24V"
- board text added: "5V"
- board text added: "GND"
- board text added: "JLCJLCJLCJLC"
- board text added: "Sherline CNC Input Board - Rev A"
- board text added: "© 2021 A.C. Wright Design | acwrightdesign.com"

Commit message: Add Rev B
Parts:
- H1, H2, H3, H4, H5: value MountingHole -> MountingHole_Pad
- J12: value Encoder -> Encoder Input
- J14: value Encoder -> Encoder Output
- J2: footprint TerminalBlock_Phoenix:TerminalBlock_Phoenix_PT-1,5-3-5.0-H_1x03_P5.00mm_Horizontal -> TerminalBlock_Phoenix:TerminalBlock_Phoenix_PT-1,5-4-5.0-H_1x04_P5.00mm_Horizontal
- moved J14 10.2 mm to (90.0, 127.0)
- moved J4 10.2 mm to (72.5, 57.3)
- moved J8 10.2 mm to (66.0, 58.0)
- moved G*** 10.2 mm to (60.0, 112.5)
- moved H1 10.2 mm to (58.0, 46.0)
- moved H2 10.2 mm to (58.0, 134.0)
- moved H3 10.2 mm to (226.0, 134.0)
- moved H4 10.2 mm to (226.0, 46.0)
- moved H5 10.2 mm to (151.0, 108.0)
- moved J1 10.2 mm to (171.5, 58.5)
- moved J10 10.2 mm to (66.0, 84.0)
- moved J11 10.2 mm to (66.0, 97.0)
- moved J12 10.2 mm to (90.0, 113.7)
- moved J13 10.2 mm to (206.8, 93.5)
- moved J15 10.2 mm to (225.5, 98.0)
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Connections:
- J2 pad 3: 24V -> 12V
- J3 pad 2: 5V -> 12V
Routing:
- net 12V: track 0.00 -> 180.1 mm, vias 0 -> 2
- net 5V: track 189.8 -> 121.7 mm, vias 1 -> 0
- net Net-(J1-Pad20): track 119.8 -> 131.1 mm
- net 24V: track 221.4 -> 220.1 mm
Other:
- board text added: "12V"
- board text added: "Sherline CNC Input Board - Rev B"
- board text removed: "Sherline CNC Input Board - Rev A"
