File: Hardware/Input Board/Input Board.kicad_sch (KiCad schematic)
At the start: 30 parts, among them J1 Relay, J10 Y Limit, J11 Z Limit, J12 Probe, J13 A Input, J14 Z Input, J15 Y Input, J16 X Input, J17 X Output, J18 Y Output, J19 Z Output, J2 24V, J20 A Output, J3 LED Lights, J4 Mist, J5 Motor Board, J6 Encoder Input, J7 Accessory, J8 Encoder Output, J9 X Limit, K1 SRD-24VDC-SL-C, K2 SRD-24VDC-SL-C

Commit message: Library cleanup
Parts:
- H1, H2, H3, H4: footprint (none) -> MountingHole:MountingHole_3.2mm_M3
- J1: footprint (none) -> Connector_Dsub:DSUB-25_Female_Vertical_P2.77x2.84mm_MountingHoles
- J13, J14, J15, J16, J6, J7: footprint (none) -> Connector_Dsub:DSUB-9_Female_Vertical_P2.77x2.84mm_MountingHoles
- J17, J18, J19, J20, J5: footprint (none) -> DIN5-RA-PTH:DIN5-RA-PTH
- J2: footprint (none) -> TerminalBlock_Phoenix:TerminalBlock_Phoenix_PT-1,5-2-5.0-H_1x02_P5.00mm_Horizontal
- J3: footprint (none) -> Connector_BarrelJack:BarrelJack_Horizontal
- J8: footprint (none) -> Connector_Dsub:DSUB-9_Female_Horizontal_P2.77x2.84mm_EdgePinOffset9.90mm_Housed_MountingHolesOffset11.32mm
- K1, K2: footprint Input Board:SRD-24VDC-SL-C -> SRD-24VDC-SL-C:SRD-24VDC-SL-C
- R1, R2, R3, R4: footprint (none) -> Resistor_THT:R_Axial_DIN0411_L9.9mm_D3.6mm_P15.24mm_Horizontal

Commit message: Finish schematics
Parts:
- removed J2: 24V, TerminalBlock_Phoenix:TerminalBlock_Phoenix_PT-1,5-2-5.0-H_1x02_P5.00mm_Horizontal, symbol Connector:Screw_Terminal_01x02
- removed J4: Mist, symbol Connector:AudioJack3
- removed J5: Motor Board, DIN5-RA-PTH:DIN5-RA-PTH, symbol Connector:DIN-5
- removed K1, K2: SRD-24VDC-SL-C, SRD-24VDC-SL-C:SRD-24VDC-SL-C, symbol SRD-24VDC-SL-C:SRD-24VDC-SL-C
- added J10: Flood, Connector_BarrelJack:BarrelJack_Horizontal, symbol Connector:Barrel_Jack
- added J11: Other, Connector_BarrelJack:BarrelJack_Horizontal, symbol Connector:Barrel_Jack
- added J2: Power, symbol Connector:Screw_Terminal_01x03
- added J3: Motor Board, Connector_RJ:RJ45_Amphenol_54602-x08_Horizontal, symbol Connector:RJ45
- added J4, J5, J6, J7: Conn_01x02, symbol Connector_Generic:Conn_01x02
- added J9: Mist, Connector_BarrelJack:BarrelJack_Horizontal, symbol Connector:Barrel_Jack
- added K1, K2, K3, K4: SRD-05VDC-SL-C, SRD-05VDC-SL-C:SRD-05VDC-SL-C, symbol SRD05VDC-SL-C:SRD-05VDC-SL-C
- J1: value Relay -> Relays
- J13: renamed from J7; value Accessory -> Signals
- J8: renamed from J3; value LED Lights -> Lamp
- renumbered J6 to J12, J8 to J14, J9 to J15, J10 to J16, J11 to J17, J12 to J18, J13 to J19, J14 to J20, J15 to J21, J16 to J22, J17 to J23, J18 to J24, J19 to J25, J20 to J26
Connections:
- net FWD: now also J1.3, J3.5; no longer J1.4
- net GND: now also J10.2, J11.2, J2.1 (Pin_1), J3.1, J9.2, K1.A2, K2.A2, K3.A2, K4.A2
- net REV: now also J1.17 (P17), J3.4; no longer J1.5
- net SPINDLE_0_10V: now also J3.8
- net 5V: now reaches J1.10
- net 5V: now also J1.18 (P18), J1.21 (P21), J1.7, J2.2 (Pin_2), J3.2
- net at J1.20 (P20): now also K2.A1
- net at J1.23 (P23): now also K4.A1
- net at J1.6: now also K1.A1
- net at J1.9: now also K3.A1
- net at J8.1: now also J4.1 (Pin_1), K1.NO
- removed net +24V: J1.14 (P14), J1.17 (P17), J1.3
- net LAMP: no longer names the net of J1.1
- net MIST renamed FWD_REV_COM
- net FWD_REV_COM: now also J1.4, J3.3
- net SPINDLE_GND renamed SPINDLE_COM
- net SPINDLE_COM: now also J3.7
- new net: J5.2 (Pin_2), K2.NC
- new net: J5.1 (Pin_1), J9.1, K2.NO
- new net: J6.2 (Pin_2), K3.NC
- new net: J10.1, J6.1 (Pin_1), K3.NO
- new net: J4.2 (Pin_2), K1.NC
- new net: J11.1, J7.1 (Pin_1), K4.NO
- new net: J7.2 (Pin_2), K4.NC
- new net 24V: J2.3 (Pin_3), J3.6, K1.COM, K2.COM, K3.COM, K4.COM
- no-connect marks 37 -> 29
Other:
- moved on the sheet: J1, J12, J13, J14, J15, J16, J17, J18, J8

Commit message: Add missing footprints
Parts:
- J15, J16, J17, J18: footprint (none) -> PJ-307:PJ-307-3
- J2: footprint (none) -> TerminalBlock_Phoenix:TerminalBlock_Phoenix_PT-1,5-3-5.0-H_1x03_P5.00mm_Horizontal
- J4, J5, J6, J7: footprint (none) -> Connector_PinHeader_2.54mm:PinHeader_1x02_P2.54mm_Vertical
Changed lines of the file:
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@@
       (effects (font (size 1.27 1.27)) (justify right))
     )
-    (property "Footprint" "" (id 2) (at 171.45 57.15 0)
+    (property "Footprint" "PJ-307:PJ-307-3" (id 2) (at 171.45 57.15 0)
       (effects (font (size 1.27 1.27)) hide)
     )
@@
     (property "Reference" "J2" (id 0) (at 26.67 16.51 0))
     (property "Value" "Power" (id 1) (at 26.67 19.05 0))
-    (property "Footprint" "" (id 2) (at 26.67 25.4 0)
+    (property "Footprint" "TerminalBlock_Phoenix:TerminalBlock_Phoenix_PT-1,5-3-5.0-H_1x03_P5.00mm_Horizontal" (id 2) (at 26.67 25.4 0)
       (effects (font (size 1.27 1.27)) hide)
     )
@@
       (effects (font (size 1.27 1.27)) (justify left) hide)
     )
-    (property "Footprint" "" (id 2) (at 87.63 91.44 0)
+    (property "Footprint" "Connector_PinHeader_2.54mm:PinHeader_1x02_P2.54mm_Vertical" (id 2) (at 87.63 91.44 0)
       (effects (font (size 1.27 1.27)) hide)
     )
@@
       (effects (font (size 1.27 1.27)) (justify right))
     )
-    (property "Footprint" "" (id 2) (at 171.45 102.87 0)
+    (property "Footprint" "PJ-307:PJ-307-3" (id 2) (at 171.45 102.87 0)
       (effects (font (size 1.27 1.27)) hide)
     )
@@
       (effects (font (size 1.27 1.27)) (justify left) hide)
     )
-    (property "Footprint" "" (id 2) (at 87.63 129.54 0)
+    (property "Footprint" "Connector_PinHeader_2.54mm:PinHeader_1x02_P2.54mm_Vertical" (id 2) (at 87.63 129.54 0)
       (effects (font (size 1.27 1.27)) hide)
     )
@@
       (effects (font (size 1.27 1.27)) (justify right))
     )
-    (property "Footprint" "" (id 2) (at 171.45 87.63 0)
+    (property "Footprint" "PJ-307:PJ-307-3" (id 2) (at 171.45 87.63 0)
       (effects (font (size 1.27 1.27)) hide)
     )
@@
       (effects (font (size 1.27 1.27)) (justify right))
     )
-    (property "Footprint" "" (id 2) (at 171.45 72.39 0)
+    (property "Footprint" "PJ-307:PJ-307-3" (id 2) (at 171.45 72.39 0)
       (effects (font (size 1.27 1.27)) hide)
     )
@@
       (effects (font (size 1.27 1.27)) (justify left) hide)
     )
-    (property "Footprint" "" (id 2) (at 87.63 110.49 0)
+    (property "Footprint" "Connector_PinHeader_2.54mm:PinHeader_1x02_P2.54mm_Vertical" (id 2) (at 87.63 110.49 0)
       (effects (font (size 1.27 1.27)) hide)
     )
@@
       (effects (font (size 1.27 1.27)) (justify left) hide)
     )
-    (property "Footprint" "" (id 2) (at 87.63 148.59 0)
+    (property "Footprint" "Connector_PinHeader_2.54mm:PinHeader_1x02_P2.54mm_Vertical" (id 2) (at 87.63 148.59 0)
       (effects (font (size 1.27 1.27)) hide)
     )
@@
     )
     (path "/6bc5ed5b-f9f0-4b08-aea8-cdc49245ad26"
-      (reference "J2") (unit 1) (value "Power") (footprint "")
+      (reference "J2") (unit 1) (value "Power") (footprint "TerminalBlock_Phoenix:TerminalBlock_Phoenix_PT-1,5-3-5.0-H_1x03_P5.00mm_Horizontal")
     )
     (path "/384947f5-272c-42b4-9b6a-6efa993dfbb1"
@@
     )
     (path "/6d72ec54-0c84-4307-ba30-529b224a9303"
-      (reference "J4") (unit 1) (value "Conn_01x02") (footprint "")
+      (reference "J4") (unit 1) (value "Conn_01x02") (footprint "Connector_PinHeader_2.54mm:PinHeader_1x02_P2.54mm_Vertical")
     )
     (path "/ad618a0d-6db7-4aad-846a-f34d6c29d610"
-      (reference "J5") (unit 1) (value "Conn_01x02") (footprint "")
+      (reference "J5") (unit 1) (value "Conn_01x02") (footprint "Connector_PinHeader_2.54mm:PinHeader_1x02_P2.54mm_Vertical")
     )
     (path "/95f497d5-b5ca-4c89-af6d-162da4cfe728"
-      (reference "J6") (unit 1) (value "Conn_01x02") (footprint "")
+      (reference "J6") (unit 1) (value "Conn_01x02") (footprint "Connector_PinHeader_2.54mm:PinHeader_1x02_P2.54mm_Vertical")
     )
     (path "/f0efd7d9-5329-435f-b120-2377b48fb3c9"
-      (reference "J7") (unit 1) (value "Conn_01x02") (footprint "")
+      (reference "J7") (unit 1) (value "Conn_01x02") (footprint "Connector_PinHeader_2.54mm:PinHeader_1x02_P2.54mm_Vertical")
     )
     (path "/7e1ce275-b722-4915-98ee-90aaed1e90bb"
@@
     )
     (path "/58de89d8-d543-44a1-b82f-809d3e66778c"
-      (reference "J15") (unit 1) (value "X Limit") (footprint "")
+      (reference "J15") (unit 1) (value "X Limit") (footprint "PJ-307:PJ-307-3")
     )
     (path "/ad042fdc-3831-4d29-b8a5-eabf98c86236"
-      (reference "J16") (unit 1) (value "Y Limit") (footprint "")
+      (reference "J16") (unit 1) (value "Y Limit") (footprint "PJ-307:PJ-307-3")
     )
     (path "/9ffef121-5a7e-443e-b69b-7539e2966335"
-      (reference "J17") (unit 1) (value "Z Limit") (footprint "")
+      (reference "J17") (unit 1) (value "Z Limit") (footprint "PJ-307:PJ-307-3")
     )
     (path "/91273a26-67a0-43d8-8439-59b7763f5daf"
-      (reference "J18") (unit 1) (value "Probe") (footprint "")
+      (reference "J18") (unit 1) (value "Probe") (footprint "PJ-307:PJ-307-3")
     )
     (path "/4ee888ad-4270-427b-a769-7c30ad6e1868"

Commit message: Update
Parts:
- added H5: MountingHole_Pad, MountingHole:MountingHole_3.2mm_M3, symbol Mechanical:MountingHole
- H1, H2, H3, H4: symbol Mechanical:MountingHole_Pad -> Mechanical:MountingHole
- J1: symbol Connector:DB25_Female_MountingHoles -> Connector:DB25_Female
- J12, J13, J14: symbol Connector:DB9_Female_MountingHoles -> Connector:DB9_Female
- J19: value A Input -> X Input; symbol Connector:DB9_Female_MountingHoles -> Connector:DB9_Female
- J20: value Z Input -> Y Input; symbol Connector:DB9_Female_MountingHoles -> Connector:DB9_Female
- J21: value Y Input -> Z Input; symbol Connector:DB9_Female_MountingHoles -> Connector:DB9_Female
- J22: value X Input -> A Input; symbol Connector:DB9_Female_MountingHoles -> Connector:DB9_Female
Connections:
- removed net Earth: H1.1, H2.1, H3.1, H4.1, J1.0 (PAD), J12.0 (PAD), J13.0 (PAD), J14.0 (PAD), J19.0 (PAD), J20.0 (PAD), J21.0 (PAD), J22.0 (PAD)

Commit message: Rev A boards ordered
Other:
- title: Sherline CNC Conversion - Input Board -> Sherline CNC - Input Board
Changed lines of the file:
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@@
   (paper "A4")
   (title_block
-    (title "Sherline CNC Conversion - Input Board")
+    (title "Sherline CNC - Input Board")
     (date "2021-11-28")
     (rev "A")

Commit message: Add Rev B
Parts:
- J2: footprint TerminalBlock_Phoenix:TerminalBlock_Phoenix_PT-1,5-3-5.0-H_1x03_P5.00mm_Horizontal -> TerminalBlock_Phoenix:TerminalBlock_Phoenix_PT-1,5-4-5.0-H_1x04_P5.00mm_Horizontal; symbol Connector:Screw_Terminal_01x03 -> Connector:Screw_Terminal_01x04
Connections:
- net 24V: now also J2.4 (Pin_4); no longer J2.3 (Pin_3)
- net 5V: no longer J3.2
- new net 12V: J2.3 (Pin_3), J3.2
Changed lines of the file:
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@@
   (title_block
     (title "Sherline CNC - Input Board")
-    (date "2021-11-28")
-    (rev "A")
+    (date "2022-02-10")
+    (rev "B")
     (company "A.C. Wright Design")
   )
@@
   (junction (at 34.29 30.48) (diameter 0) (color 0 0 0 0)
   )
-  (junction (at 78.74 22.86) (diameter 0) (color 0 0 0 0)
+  (junction (at 53.34 22.86) (diameter 0) (color 0 0 0 0)
   )
   (junction (at 40.64 76.2) (diameter 0) (color 0 0 0 0)
@@
   )
   (junction (at 53.34 105.41) (diameter 0) (color 0 0 0 0)
+  )
+  (junction (at 78.74 20.32) (diameter 0) (color 0 0 0 0)
   )
   (junction (at 95.25 116.84) (diameter 0) (color 0 0 0 0)
@@
     (stroke (width 0) (type default) (color 0 0 0 0))
   )
+  (wire (pts (xy 53.34 22.86) (xy 58.42 22.86))
+    (stroke (width 0) (type default) (color 0 0 0 0))
+  )
   (wire (pts (xy 40.64 25.4) (xy 40.64 30.48))
     (stroke (width 0) (type default) (color 0 0 0 0))
@@
     (stroke (width 0) (type default) (color 0 0 0 0))
   )
+  (wire (pts (xy 31.75 22.86) (xy 53.34 22.86))
+    (stroke (width 0) (type default) (color 0 0 0 0))
+  )
   (wire (pts (xy 72.39 143.51) (xy 85.09 143.51))
     (stroke (width 0) (type default) (color 0 0 0 0))
@@
     (stroke (width 0) (type default) (color 0 0 0 0))
   )
-  (wire (pts (xy 78.74 22.86) (xy 83.82 22.86))
+  (wire (pts (xy 78.74 20.32) (xy 83.82 20.32))
     (stroke (width 0) (type default) (color 0 0 0 0))
   )
@@
     (stroke (width 0) (type default) (color 0 0 0 0))
   )
+  (wire (pts (xy 31.75 20.32) (xy 78.74 20.32))
+    (stroke (width 0) (type default) (color 0 0 0 0))
+  )
   (wire (pts (xy 129.54 161.29) (xy 142.24 161.29))
     (stroke (width 0) (type default) (color 0 0 0 0))
@@
     (stroke (width 0) (type default) (color 0 0 0 0))
   )
-  (wire (pts (xy 78.74 22.86) (xy 78.74 30.48))
+  (wire (pts (xy 78.74 20.32) (xy 78.74 30.48))
     (stroke (width 0) (type default) (color 0 0 0 0))
   )
@@
   )
   (wire (pts (xy 53.34 124.46) (xy 53.34 143.51))
-    (stroke (width 0) (type default) (color 0 0 0 0))
-  )
-  (wire (pts (xy 31.75 22.86) (xy 78.74 22.86))
     (stroke (width 0) (type default) (color 0 0 0 0))
   )
@@
     )
   )
-  (global_label "5V" (shape input) (at 40.64 182.88 0) (fields_autoplaced)
+  (global_label "12V" (shape input) (at 40.64 182.88 0) (fields_autoplaced)
     (effects (font (size 1.27 1.27)) (justify left))
-    (property "Intersheet References" "${INTERSHEET_REFS}" (id 0) (at 45.2623 182.8006 0)
+    (property "Intersheet References" "${INTERSHEET_REFS}" (id 0) (at 46.4718 182.8006 0)
       (effects (font (size 1.27 1.27)) (justify left) hide)
     )
@@
     )
   )
-  (global_label "24V" (shape output) (at 83.82 22.86 0) (fields_autoplaced)
+  (global_label "24V" (shape output) (at 83.82 20.32 0) (fields_autoplaced)
     (effects (font (size 1.27 1.27)) (justify left))
-    (property "Intersheet References" "${INTERSHEET_REFS}" (id 0) (at 89.6518 22.7806 0)
+    (property "Intersheet References" "${INTERSHEET_REFS}" (id 0) (at 89.6518 20.2406 0)
       (effects (font (size 1.27 1.27)) (justify left) hide)
     )
@@
     (effects (font (size 1.27 1.27)) (justify left))
     (property "Intersheet References" "${INTERSHEET_REFS}" (id 0) (at 50.2818 71.0406 0)
+      (effects (font (size 1.27 1.27)) (justify left) hide)
+    )
+  )
+  (global_label "12V" (shape output) (at 58.42 22.86 0) (fields_autoplaced)
+    (effects (font (size 1.27 1.27)) (justify left))
+    (property "Intersheet References" "${INTERSHEET_REFS}" (id 0) (at 64.2518 22.7806 0)
       (effects (font (size 1.27 1.27)) (justify left) hide)
     )
@@
     (pin "2")
   )
-  (symbol (lib_id "Connector:Screw_Terminal_01x03") (at 26.67 25.4 180) (unit 1)
-    (in_bom yes) (on_board yes) (fields_autoplaced)
-    (property "Reference" "J2" (id 0) (at 26.67 16.51 0))
-    (property "Value" "Power" (id 1) (at 26.67 19.05 0))
-    (property "Footprint" "TerminalBlock_Phoenix:TerminalBlock_Phoenix_PT-1,5-3-5.0-H_1x03_P5.00mm_Horizontal" (id 2) (at 26.67 25.4 0)
+  (symbol (lib_id "Connector:Screw_Terminal_01x04") (at 26.67 25.4 180) (unit 1)
+    (in_bom yes) (on_board yes)
+    (property "Reference" "J2" (id 0) (at 26.67 15.24 0))
+    (property "Value" "Power" (id 1) (at 26.67 17.78 0))
+    (property "Footprint" "TerminalBlock_Phoenix:TerminalBlock_Phoenix_PT-1,5-4-5.0-H_1x04_P5.00mm_Horizontal" (id 2) (at 26.67 25.4 0)
       (effects (font (size 1.27 1.27)) hide)
     )
@@
     (pin "2")
     (pin "3")
+    (pin "4")
   )
   (symbol (lib_id "Connector_Generic:Conn_01x02") (at 87.63 91.44 270) (unit 1)
@@
     (pin "2")
   )
+  (symbol (lib_id "power:PWR_FLAG") (at 53.34 22.86 180) (unit 1)
+    (in_bom yes) (on_board yes) (fields_autoplaced)
+    (property "Reference" "#FLG01" (id 0) (at 53.34 24.765 0)
+      (effects (font (size 1.27 1.27)) hide)
+    )
+    (property "Value" "PWR_FLAG" (id 1) (at 53.3399 26.67 90)
+      (effects (font (size 1.27 1.27)) (justify left) hide)
+    )
+    (property "Footprint" "" (id 2) (at 53.34 22.86 0)
+      (effects (font (size 1.27 1.27)) hide)
+    )
+    (property "Datasheet" "~" (id 3) (at 53.34 22.86 0)
+      (effects (font (size 1.27 1.27)) hide)
+    )
+    (pin "1")
+  )
   (symbol (lib_id "Device:R") (at 219.71 130.81 90) (mirror x) (unit 1)
     (in_bom yes) (on_board yes) (fields_autoplaced)
@@
   )
   (symbol_instances
+    (path "/b1ee7b76-88f6-42aa-8359-17590ed83a50"
+      (reference "#FLG01") (unit 1) (value "PWR_FLAG") (footprint "")
+    )
     (path "/d32037e5-ca9f-4403-a040-cb7d43e0fe17"
       (reference "#FLG02") (unit 1) (value "PWR_FLAG") (footprint "")
@@
     )
     (path "/6bc5ed5b-f9f0-4b08-aea8-cdc49245ad26"
-      (reference "J2") (unit 1) (value "Power") (footprint "TerminalBlock_Phoenix:TerminalBlock_Phoenix_PT-1,5-3-5.0-H_1x03_P5.00mm_Horizontal")
+      (reference "J2") (unit 1) (value "Power") (footprint "TerminalBlock_Phoenix:TerminalBlock_Phoenix_PT-1,5-4-5.0-H_1x04_P5.00mm_Horizontal")
     )
     (path "/384947f5-272c-42b4-9b6a-6efa993dfbb1"
