File: Hardware/Motor Board/Motor Board.kicad_sch (KiCad schematic)
At the start: 10 parts, among them J2 Conn_02x06_Counter_Clockwise, J4 Screw_Terminal_01x03, J5 DIN-5, J8 Screw_Terminal_01x05, K1 SRD-24VDC-SL-C, K2 SRD-24VDC-SL-C, K3 SRD-24VDC-SL-C, K4 SRD-24VDC-SL-C

Commit message: Library cleanup
Parts:
- added H1, H2, H3, H4: MountingHole, symbol Mechanical:MountingHole
- J1: renamed from J4; footprint (none) -> TerminalBlock_Phoenix:TerminalBlock_Phoenix_PT-1,5-3-5.0-H_1x03_P5.00mm_Horizontal
- J2: renamed from J5; footprint (none) -> Motor Board:DIN5-RA-PTH
- J4: renamed from J?; footprint (none) -> TerminalBlock_Phoenix:TerminalBlock_Phoenix_PT-1,5-2-5.0-H_1x02_P5.00mm_Horizontal
- J5: renamed from J?; footprint (none) -> TerminalBlock_Phoenix:TerminalBlock_Phoenix_PT-1,5-4-5.0-H_1x04_P5.00mm_Horizontal
- J6: renamed from J8; footprint (none) -> TerminalBlock_Phoenix:TerminalBlock_Phoenix_PT-1,5-5-5.0-H_1x05_P5.00mm_Horizontal
- renumbered J2 to J3
Changed lines of the file:
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@@
+    )
+  )
+  (symbol (lib_id "Mechanical:MountingHole") (at 72.39 166.37 0) (unit 1)
+    (in_bom yes) (on_board yes) (fields_autoplaced)
+    (property "Reference" "H1" (id 0) (at 74.93 165.0999 0)
+      (effects (font (size 1.27 1.27)) (justify left))
+    )
+    (property "Value" "MountingHole" (id 1) (at 74.93 167.6399 0)
+      (effects (font (size 1.27 1.27)) (justify left))
+    )
+    (property "Footprint" "" (id 2) (at 72.39 166.37 0)
+      (effects (font (size 1.27 1.27)) hide)
+    )
+    (property "Datasheet" "~" (id 3) (at 72.39 166.37 0)
+      (effects (font (size 1.27 1.27)) hide)
+    )
+  )
+  (symbol (lib_id "Mechanical:MountingHole") (at 72.39 177.8 0) (unit 1)
+    (in_bom yes) (on_board yes) (fields_autoplaced)
+    (property "Reference" "H2" (id 0) (at 74.93 176.5299 0)
+      (effects (font (size 1.27 1.27)) (justify left))
+    )
+    (property "Value" "MountingHole" (id 1) (at 74.93 179.0699 0)
+      (effects (font (size 1.27 1.27)) (justify left))
+    )
+    (property "Footprint" "" (id 2) (at 72.39 177.8 0)
+      (effects (font (size 1.27 1.27)) hide)
+    )
+    (property "Datasheet" "~" (id 3) (at 72.39 177.8 0)
+      (effects (font (size 1.27 1.27)) hide)
     )
   )
   (symbol (lib_id "Connector:Screw_Terminal_01x04") (at 175.26 54.61 0) (unit 1)
     (in_bom yes) (on_board yes)
-    (property "Reference" "J?" (id 0) (at 177.8 54.6099 0)
+    (property "Reference" "J5" (id 0) (at 177.8 54.6099 0)
       (effects (font (size 1.27 1.27)) (justify left))
     )
@@
       (effects (font (size 1.27 1.27)) (justify left))
     )
-    (property "Footprint" "" (id 2) (at 175.26 54.61 0)
+    (property "Footprint" "TerminalBlock_Phoenix:TerminalBlock_Phoenix_PT-1,5-4-5.0-H_1x04_P5.00mm_Horizontal" (id 2) (at 175.26 54.61 0)
       (effects (font (size 1.27 1.27)) hide)
     )
@@
   (symbol (lib_id "Connector:DIN-5") (at 77.47 113.03 180) (unit 1)
     (in_bom yes) (on_board yes)
-    (property "Reference" "J5" (id 0) (at 77.4699 102.87 0))
+    (property "Reference" "J2" (id 0) (at 77.4699 102.87 0))
     (property "Value" "DIN-5" (id 1) (at 77.4699 105.41 0))
-    (property "Footprint" "" (id 2) (at 77.47 113.03 0)
+    (property "Footprint" "Motor Board:DIN5-RA-PTH" (id 2) (at 77.47 113.03 0)
       (effects (font (size 1.27 1.27)) hide)
     )
@@
     (pin "5")
   )
+  (symbol (lib_id "Mechanical:MountingHole") (at 95.25 166.37 0) (unit 1)
+    (in_bom yes) (on_board yes) (fields_autoplaced)
+    (property "Reference" "H3" (id 0) (at 97.79 165.0999 0)
+      (effects (font (size 1.27 1.27)) (justify left))
+    )
+    (property "Value" "MountingHole" (id 1) (at 97.79 167.6399 0)
+      (effects (font (size 1.27 1.27)) (justify left))
+    )
+    (property "Footprint" "" (id 2) (at 95.25 166.37 0)
+      (effects (font (size 1.27 1.27)) hide)
+    )
+    (property "Datasheet" "~" (id 3) (at 95.25 166.37 0)
+      (effects (font (size 1.27 1.27)) hide)
+    )
+  )
   (symbol (lib_id "Connector:Screw_Terminal_01x05") (at 175.26 80.01 0) (unit 1)
     (in_bom yes) (on_board yes)
-    (property "Reference" "J8" (id 0) (at 177.8 78.7399 0)
+    (property "Reference" "J6" (id 0) (at 177.8 78.7399 0)
       (effects (font (size 1.27 1.27)) (justify left))
     )
@@
       (effects (font (size 1.27 1.27)) (justify left))
     )
-    (property "Footprint" "" (id 2) (at 175.26 80.01 0)
+    (property "Footprint" "TerminalBlock_Phoenix:TerminalBlock_Phoenix_PT-1,5-5-5.0-H_1x05_P5.00mm_Horizontal" (id 2) (at 175.26 80.01 0)
       (effects (font (size 1.27 1.27)) hide)
     )
@@
   (symbol (lib_id "Connector_Generic:Conn_02x06_Counter_Clockwise") (at 80.01 49.53 0) (unit 1)
     (in_bom yes) (on_board yes)
-    (property "Reference" "J2" (id 0) (at 81.28 38.1 0))
+    (property "Reference" "J3" (id 0) (at 81.28 38.1 0))
     (property "Value" "Conn_02x06_Counter_Clockwise" (id 1) (at 81.28 40.64 0))
     (property "Footprint" "Connector_Molex:Molex_Micro-Fit_3.0_43045-1200_2x06_P3.00mm_Horizontal" (id 2) (at 80.01 49.53 0)
@@
   (symbol (lib_id "Connector:Screw_Terminal_01x02") (at 175.26 34.29 0) (unit 1)
     (in_bom yes) (on_board yes)
-    (property "Reference" "J?" (id 0) (at 177.8 34.2899 0)
+    (property "Reference" "J4" (id 0) (at 177.8 34.2899 0)
       (effects (font (size 1.27 1.27)) (justify left))
     )
@@
       (effects (font (size 1.27 1.27)) (justify left))
     )
-    (property "Footprint" "" (id 2) (at 175.26 34.29 0)
+    (property "Footprint" "TerminalBlock_Phoenix:TerminalBlock_Phoenix_PT-1,5-2-5.0-H_1x02_P5.00mm_Horizontal" (id 2) (at 175.26 34.29 0)
       (effects (font (size 1.27 1.27)) hide)
     )
@@
   (symbol (lib_id "Connector:Screw_Terminal_01x03") (at 76.2 86.36 180) (unit 1)
     (in_bom yes) (on_board yes)
-    (property "Reference" "J4" (id 0) (at 76.2 77.47 0))
+    (property "Reference" "J1" (id 0) (at 76.2 77.47 0))
     (property "Value" "Screw_Terminal_01x03" (id 1) (at 76.2 80.01 0))
-    (property "Footprint" "" (id 2) (at 76.2 86.36 0)
+    (property "Footprint" "TerminalBlock_Phoenix:TerminalBlock_Phoenix_PT-1,5-3-5.0-H_1x03_P5.00mm_Horizontal" (id 2) (at 76.2 86.36 0)
       (effects (font (size 1.27 1.27)) hide)
     )
@@
     (pin "NO")
   )
+  (symbol (lib_id "Mechanical:MountingHole") (at 95.25 177.8 0) (unit 1)
+    (in_bom yes) (on_board yes) (fields_autoplaced)
+    (property "Reference" "H4" (id 0) (at 97.79 176.5299 0)
+      (effects (font (size 1.27 1.27)) (justify left))
+    )
+    (property "Value" "MountingHole" (id 1) (at 97.79 179.0699 0)
+      (effects (font (size 1.27 1.27)) (justify left))
+    )
+    (property "Footprint" "" (id 2) (at 95.25 177.8 0)
+      (effects (font (size 1.27 1.27)) hide)
+    )
+    (property "Datasheet" "~" (id 3) (at 95.25 177.8 0)
+      (effects (font (size 1.27 1.27)) hide)
+    )
+  )
   (sheet_instances
     (path "/" (page "1"))
   )
   (symbol_instances
+    (path "/0dbe3354-4a8d-4b3a-bc97-120b726e6b74"
+      (reference "H1") (unit 1) (value "MountingHole") (footprint "")
+    )
+    (path "/1ba443a3-27eb-47ab-a61d-72bb20dc6d95"
+      (reference "H2") (unit 1) (value "MountingHole") (footprint "")
+    )
+    (path "/7565e19c-aec2-4922-88dc-879db68f5c1c"
+      (reference "H3") (unit 1) (value "MountingHole") (footprint "")
+    )
+    (path "/fb94f691-33d3-4c5b-bd7d-f9acacd56ae9"
+      (reference "H4") (unit 1) (value "MountingHole") (footprint "")
+    )
+    (path "/c937db2f-65df-4632-a408-313f48ab950d"
+      (reference "J1") (unit 1) (value "Screw_Terminal_01x03") (footprint "TerminalBlock_Phoenix:TerminalBlock_Phoenix_PT-1,5-3-5.0-H_1x03_P5.00mm_Horizontal")
+    )
+    (path "/485c68c6-5094-4829-bd33-1132c569abec"
+      (reference "J2") (unit 1) (value "DIN-5") (footprint "Motor Board:DIN5-RA-PTH")
+    )
     (path "/7d9513ef-5bc9-4157-b475-9f1f0ac4642b"
-      (reference "J2") (unit 1) (value "Conn_02x06_Counter_Clockwise") (footprint "Connector_Molex:Molex_Micro-Fit_3.0_43045-1200_2x06_P3.00mm_Horizontal")
-    )
-    (path "/c937db2f-65df-4632-a408-313f48ab950d"
-      (reference "J4") (unit 1) (value "Screw_Terminal_01x03") (footprint "")
-    )
-    (path "/485c68c6-5094-4829-bd33-1132c569abec"
-      (reference "J5") (unit 1) (value "DIN-5") (footprint "")
+      (reference "J3") (unit 1) (value "Conn_02x06_Counter_Clockwise") (footprint "Connector_Molex:Molex_Micro-Fit_3.0_43045-1200_2x06_P3.00mm_Horizontal")
+    )
+    (path "/c267333c-9591-4aca-9d90-0e4ddcc2f0a3"
+      (reference "J4") (unit 1) (value "Screw_Terminal_01x02") (footprint "TerminalBlock_Phoenix:TerminalBlock_Phoenix_PT-1,5-2-5.0-H_1x02_P5.00mm_Horizontal")
+    )
+    (path "/210de7fe-5340-454f-beaa-46a403c519b5"
+      (reference "J5") (unit 1) (value "Screw_Terminal_01x04") (footprint "TerminalBlock_Phoenix:TerminalBlock_Phoenix_PT-1,5-4-5.0-H_1x04_P5.00mm_Horizontal")
     )
     (path "/76587127-3eb0-4b30-b202-b079a965a91d"
-      (reference "J8") (unit 1) (value "Screw_Terminal_01x05") (footprint "")
-    )
-    (path "/210de7fe-5340-454f-beaa-46a403c519b5"
-      (reference "J?") (unit 1) (value "Screw_Terminal_01x04") (footprint "")
-    )
-    (path "/c267333c-9591-4aca-9d90-0e4ddcc2f0a3"
-      (reference "J?") (unit 1) (value "Screw_Terminal_01x02") (footprint "")
+      (reference "J6") (unit 1) (value "Screw_Terminal_01x05") (footprint "TerminalBlock_Phoenix:TerminalBlock_Phoenix_PT-1,5-5-5.0-H_1x05_P5.00mm_Horizontal")
     )
     (path "/9d3f9f4c-7782-4db3-8daa-0d892f9d3e1b"

Commit message: Finish schematics
Parts:
- removed J2: DIN-5, Motor Board:DIN5-RA-PTH, symbol Connector:DIN-5
- removed J3: Conn_02x06_Counter_Clockwise, Connector_Molex:Molex_Micro-Fit_3.0_43045-1200_2x06_P3.00mm_Horizontal, symbol Connector_Generic:Conn_02x06_Counter_Clockwise
- removed K1, K2, K3, K4: SRD-24VDC-SL-C, Motor Board:SRD-24VDC-SL-C, symbol SRD-24VDC-SL-C:SRD-24VDC-SL-C
- added A1: Arduino_Nano_v3.x, Module:Arduino_Nano, symbol MCU_Module:Arduino_Nano_v3.x
- added D1, D2, D3, D4, D5: 1N4007, Diode_THT:D_DO-41_SOD81_P10.16mm_Horizontal, symbol Diode:1N4007
- added J1: Input Board, Connector_RJ:RJ45_Amphenol_54602-x08_Horizontal, symbol Connector:RJ45
- added J3: Power, TerminalBlock_Phoenix:TerminalBlock_Phoenix_PT-1,5-3-5.0-H_1x03_P5.00mm_Horizontal, symbol Connector:Screw_Terminal_01x03
- added J4: Indicator LED, TerminalBlock_Phoenix:TerminalBlock_Phoenix_PT-1,5-2-5.0-H_1x02_P5.00mm_Horizontal, symbol Connector:Screw_Terminal_01x02
- added J5: Auto / Fwd / Rev, TerminalBlock_Phoenix:TerminalBlock_Phoenix_PT-1,5-3-5.0-H_1x03_P5.00mm_Horizontal, symbol Connector:Screw_Terminal_01x03
- added J6: Direction LED (Bi-Color), TerminalBlock_Phoenix:TerminalBlock_Phoenix_PT-1,5-2-5.0-H_1x02_P5.00mm_Horizontal, symbol Connector:Screw_Terminal_01x02
- added K1, K2, K3, K4, K5: SRD-05VDC-SL-C, SRD-05VDC-SL-C:SRD-05VDC-SL-C, symbol SRD05VDC-SL-C:SRD-05VDC-SL-C
- added Q1, Q2, Q3, Q4, Q5: 2N2222, Package_TO_SOT_THT:TO-92L_HandSolder, symbol Device:Q_NPN_CBE
- added R1, R2, R3, R4: 10K, Resistor_THT:R_Axial_DIN0309_L9.0mm_D3.2mm_P12.70mm_Horizontal, symbol Device:R
- added R10, R6, R7, R8, R9: 1K, Resistor_THT:R_Axial_DIN0309_L9.0mm_D3.2mm_P12.70mm_Horizontal, symbol Device:R
- added R5: 330, Resistor_THT:R_Axial_DIN0309_L9.0mm_D3.2mm_P12.70mm_Horizontal, symbol Device:R
- H1, H2, H3, H4: footprint (none) -> MountingHole:MountingHole_3.2mm_M3
- J2: renamed from J1; value Screw_Terminal_01x03 -> Speed; Label Speed (5K) -> (none)
- J7: renamed from J4; value Screw_Terminal_01x02 -> Motor; Label Motor -> (none)
- J8: renamed from J5; value Screw_Terminal_01x04 -> KBLC-240D; Label KBLC-240D -> (none)
- J9: renamed from J6; value Screw_Terminal_01x05 -> KBSI-240D; Label KBSI-240D -> (none)
Connections:
- net A+: now also K2.NO, K5.NO
- net A-: now also K3.NO, K4.NO
- net FWD: now also A1.5 (D2), J1.5, R1.1
- net K5: now also J1.7
- net K6: now also K1.COM
- net M+: now also K2.COM, K4.COM
- net M-: now also K3.COM, K5.COM
- net REV: now also A1.6 (D3), J1.4, R2.1
- net KP1 renamed P1
- net SP2: no longer names the net of J2.2 (Pin_2)
- net SP2: now also K1.NO
- new net: D2.2 (A), K2.A2, Q2.1 (C)
- new net: A1.14 (D11), R5.1
- new net: J6.2 (Pin_2), R5.2
- new net: D3.2 (A), K3.A2, Q3.1 (C)
- new net: Q3.2 (B), R8.2
- new net: D5.2 (A), K5.A2, Q5.1 (C)
- new net: A1.8 (D5), J5.1 (Pin_1), R4.1
- new net: D1.2 (A), K1.A2, Q1.1 (C)
- new net: A1.7 (D4), J5.3 (Pin_3), R3.1
- new net: Q2.2 (B), R7.2
- new net: J1.8, K1.NC
- new net: D4.2 (A), K4.A2, Q4.1 (C)
- new net: Q5.2 (B), R10.2
- new net: A1.15 (D12), J6.1 (Pin_1)
- new net: Q1.2 (B), R6.2
- new net: Q4.2 (B), R9.2
- new net 24V: J1.6, J3.3 (Pin_3), J4.2 (Pin_2)
- new net 5V: A1.27 (+5V), J1.3, J5.2 (Pin_2)
- new net D10: A1.13 (D10), R10.1
- new net D6: A1.9 (D6), R6.1
- new net D7: A1.10 (D7), R7.1
- new net D8: A1.11 (D8), R8.1
- new net D9: A1.12 (D9), R9.1
- new net GND: A1.29 (GND), A1.4 (GND), J1.1, J3.1 (Pin_1), J4.1 (Pin_1), Q1.3 (E), Q2.3 (E), Q3.3 (E), Q4.3 (E), Q5.3 (E), R1.2, R2.2, R3.2, R4.2
- new net VIN: A1.30 (VIN), D1.1 (K), D2.1 (K), D3.1 (K), D4.1 (K), D5.1 (K), J1.2, J3.2 (Pin_2), K1.A1, K2.A1, K3.A1, K4.A1, K5.A1
- no-connect marks 4 -> 19
Other:
- moved on the sheet: H1, H2, H3, H4, J2, J7, J8, J9

Commit message: Add missing footprints
Parts:
- removed J4: Indicator LED, TerminalBlock_Phoenix:TerminalBlock_Phoenix_PT-1,5-2-5.0-H_1x02_P5.00mm_Horizontal, symbol Connector:Screw_Terminal_01x02
- removed J6: Direction LED (Bi-Color), TerminalBlock_Phoenix:TerminalBlock_Phoenix_PT-1,5-2-5.0-H_1x02_P5.00mm_Horizontal, symbol Connector:Screw_Terminal_01x02
- added J4: Indicator LED, Connector_PinHeader_2.54mm:PinHeader_1x02_P2.54mm_Vertical, symbol Connector_Generic:Conn_01x02
- added J6: Direction LED (Bi-Color), Connector_PinHeader_2.54mm:PinHeader_1x02_P2.54mm_Vertical, symbol Connector_Generic:Conn_01x02
- added R4, R5: 4.7K, Resistor_THT:R_Axial_DIN0309_L9.0mm_D3.2mm_P12.70mm_Horizontal, symbol Device:R
- renumbered R8 to R10, R9 to R11, R10 to R12, R4 to R6, R5 to R7, R6 to R8, R7 to R9
Connections:
- net 24V: now also R4.2, R5.2
- net GND: now also J4.1 (Pin_1)
- net at R7.2: now also J6.2 (Pin_2)
- net at A1.15 (D12): now also J6.1 (Pin_1)
- new net: J4.2 (Pin_2), R4.1, R5.1

Commit message: Update
Changed lines of the file:
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@@
     (pin "1")
+  )
+  (symbol (lib_id "A.C. Wright Logo:LOGO") (at 278.13 173.99 0) (unit 1)
+    (in_bom yes) (on_board yes) (fields_autoplaced)
+    (property "Reference" "#G1" (id 0) (at 278.13 178.2318 0)
+      (effects (font (size 1.524 1.524)) hide)
+    )
+    (property "Value" "LOGO" (id 1) (at 278.13 169.7482 0)
+      (effects (font (size 1.524 1.524)) hide)
+    )
+    (property "Footprint" "A.C. Wright Logo:A.C. Wright Logo 10mm" (id 2) (at 278.13 173.99 0)
+      (effects (font (size 1.27 1.27)) hide)
+    )
+    (property "Datasheet" "" (id 3) (at 278.13 173.99 0)
+      (effects (font (size 1.27 1.27)) hide)
+    )
   )
   (symbol (lib_id "power:GND") (at 199.39 67.31 0) (unit 1)
@@
     (pin "2")
     (pin "3")
+  )
+  (symbol (lib_id "Graphic:Logo_Open_Hardware_Small") (at 265.43 173.99 0) (unit 1)
+    (in_bom yes) (on_board yes) (fields_autoplaced)
+    (property "Reference" "#LOGO1" (id 0) (at 265.43 167.005 0)
+      (effects (font (size 1.27 1.27)) hide)
+    )
+    (property "Value" "Logo_Open_Hardware_Small" (id 1) (at 265.43 179.705 0)
+      (effects (font (size 1.27 1.27)) hide)
+    )
+    (property "Footprint" "Symbol:OSHW-Logo2_9.8x8mm_SilkScreen" (id 2) (at 265.43 173.99 0)
+      (effects (font (size 1.27 1.27)) hide)
+    )
+    (property "Datasheet" "~" (id 3) (at 265.43 173.99 0)
+      (effects (font (size 1.27 1.27)) hide)
+    )
   )
   (symbol (lib_id "SRD05VDC-SL-C:SRD-05VDC-SL-C") (at 71.12 41.91 0) (mirror y) (unit 1)
@@
       (reference "#FLG02") (unit 1) (value "PWR_FLAG") (footprint "")
     )
+    (path "/65c7b569-1517-482a-a813-3ebb49daf51a"
+      (reference "#G1") (unit 1) (value "LOGO") (footprint "A.C. Wright Logo:A.C. Wright Logo 10mm")
+    )
+    (path "/a417b009-0589-49cc-b3e0-77a45ec6f302"
+      (reference "#LOGO1") (unit 1) (value "Logo_Open_Hardware_Small") (footprint "Symbol:OSHW-Logo2_9.8x8mm_SilkScreen")
+    )
     (path "/e8e55fff-7fd3-4490-8a2d-2c7676d4e625"
