File: Hardware/Motor Board/Motor Board.kicad_sch (KiCad schematic)
At the start: 41 parts, among them J1 Input Board, J2 Speed, J3 Power, J4 Indicator LED, J5 Auto / Fwd / Rev, J6 Direction LED (Bi-Color), J7 Motor, J8 KBLC-240D, J9 KBSI-240D, K1 SRD-05VDC-SL-C, K2 SRD-05VDC-SL-C, K3 SRD-05VDC-SL-C, K4 SRD-05VDC-SL-C, K5 SRD-05VDC-SL-C, Q1 2N2222, Q2 2N2222, Q3 2N2222, Q4 2N2222, Q5 2N2222

Commit message: Rev A boards ordered
Parts:
- added H5, H6, H7: MountingHole, MountingHole:MountingHole_3.2mm_M3, symbol Mechanical:MountingHole
Other:
- title: Sherline CNC Conversion - Motor Board -> Sherline CNC - Motor Board
- moved on the sheet: H1, H2, H3, H4
Changed lines of the file:
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@@
   (paper "A4")
   (title_block
-    (title "Sherline CNC Conversion - Motor Board")
+    (title "Sherline CNC - Motor Board")
     (date "2021-11-29")
     (rev "A")
@@
     (pin "1")
   )
-  (symbol (lib_id "Mechanical:MountingHole") (at 130.81 175.26 0) (unit 1)
-    (in_bom yes) (on_board yes) (fields_autoplaced)
-    (property "Reference" "H1" (id 0) (at 133.35 173.9899 0)
-      (effects (font (size 1.27 1.27)) (justify left))
-    )
-    (property "Value" "MountingHole" (id 1) (at 133.35 176.5299 0)
-      (effects (font (size 1.27 1.27)) (justify left))
-    )
-    (property "Footprint" "MountingHole:MountingHole_3.2mm_M3" (id 2) (at 130.81 175.26 0)
-      (effects (font (size 1.27 1.27)) hide)
-    )
-    (property "Datasheet" "~" (id 3) (at 130.81 175.26 0)
+  (symbol (lib_id "Mechanical:MountingHole") (at 241.3 124.46 0) (unit 1)
+    (in_bom yes) (on_board yes) (fields_autoplaced)
+    (property "Reference" "H1" (id 0) (at 243.84 123.1899 0)
+      (effects (font (size 1.27 1.27)) (justify left))
+    )
+    (property "Value" "MountingHole" (id 1) (at 243.84 125.7299 0)
+      (effects (font (size 1.27 1.27)) (justify left))
+    )
+    (property "Footprint" "MountingHole:MountingHole_3.2mm_M3" (id 2) (at 241.3 124.46 0)
+      (effects (font (size 1.27 1.27)) hide)
+    )
+    (property "Datasheet" "~" (id 3) (at 241.3 124.46 0)
       (effects (font (size 1.27 1.27)) hide)
     )
@@
     (pin "2")
   )
-  (symbol (lib_id "Mechanical:MountingHole") (at 130.81 186.69 0) (unit 1)
-    (in_bom yes) (on_board yes) (fields_autoplaced)
-    (property "Reference" "H2" (id 0) (at 133.35 185.4199 0)
-      (effects (font (size 1.27 1.27)) (justify left))
-    )
-    (property "Value" "MountingHole" (id 1) (at 133.35 187.9599 0)
-      (effects (font (size 1.27 1.27)) (justify left))
-    )
-    (property "Footprint" "MountingHole:MountingHole_3.2mm_M3" (id 2) (at 130.81 186.69 0)
-      (effects (font (size 1.27 1.27)) hide)
-    )
-    (property "Datasheet" "~" (id 3) (at 130.81 186.69 0)
+  (symbol (lib_id "Mechanical:MountingHole") (at 241.3 135.89 0) (unit 1)
+    (in_bom yes) (on_board yes) (fields_autoplaced)
+    (property "Reference" "H2" (id 0) (at 243.84 134.6199 0)
+      (effects (font (size 1.27 1.27)) (justify left))
+    )
+    (property "Value" "MountingHole" (id 1) (at 243.84 137.1599 0)
+      (effects (font (size 1.27 1.27)) (justify left))
+    )
+    (property "Footprint" "MountingHole:MountingHole_3.2mm_M3" (id 2) (at 241.3 135.89 0)
+      (effects (font (size 1.27 1.27)) hide)
+    )
+    (property "Datasheet" "~" (id 3) (at 241.3 135.89 0)
       (effects (font (size 1.27 1.27)) hide)
     )
@@
     (pin "NO")
   )
-  (symbol (lib_id "Mechanical:MountingHole") (at 153.67 175.26 0) (unit 1)
-    (in_bom yes) (on_board yes) (fields_autoplaced)
-    (property "Reference" "H3" (id 0) (at 156.21 173.9899 0)
-      (effects (font (size 1.27 1.27)) (justify left))
-    )
-    (property "Value" "MountingHole" (id 1) (at 156.21 176.5299 0)
-      (effects (font (size 1.27 1.27)) (justify left))
-    )
-    (property "Footprint" "MountingHole:MountingHole_3.2mm_M3" (id 2) (at 153.67 175.26 0)
-      (effects (font (size 1.27 1.27)) hide)
-    )
-    (property "Datasheet" "~" (id 3) (at 153.67 175.26 0)
+  (symbol (lib_id "Mechanical:MountingHole") (at 264.16 124.46 0) (unit 1)
+    (in_bom yes) (on_board yes) (fields_autoplaced)
+    (property "Reference" "H3" (id 0) (at 266.7 123.1899 0)
+      (effects (font (size 1.27 1.27)) (justify left))
+    )
+    (property "Value" "MountingHole" (id 1) (at 266.7 125.7299 0)
+      (effects (font (size 1.27 1.27)) (justify left))
+    )
+    (property "Footprint" "MountingHole:MountingHole_3.2mm_M3" (id 2) (at 264.16 124.46 0)
+      (effects (font (size 1.27 1.27)) hide)
+    )
+    (property "Datasheet" "~" (id 3) (at 264.16 124.46 0)
       (effects (font (size 1.27 1.27)) hide)
     )
@@
     (pin "3")
   )
+  (symbol (lib_id "Mechanical:MountingHole") (at 241.3 146.05 0) (unit 1)
+    (in_bom yes) (on_board yes) (fields_autoplaced)
+    (property "Reference" "H5" (id 0) (at 243.84 144.7799 0)
+      (effects (font (size 1.27 1.27)) (justify left))
+    )
+    (property "Value" "MountingHole" (id 1) (at 243.84 147.3199 0)
+      (effects (font (size 1.27 1.27)) (justify left))
+    )
+    (property "Footprint" "MountingHole:MountingHole_3.2mm_M3" (id 2) (at 241.3 146.05 0)
+      (effects (font (size 1.27 1.27)) hide)
+    )
+    (property "Datasheet" "~" (id 3) (at 241.3 146.05 0)
+      (effects (font (size 1.27 1.27)) hide)
+    )
+  )
   (symbol (lib_id "Graphic:Logo_Open_Hardware_Small") (at 265.43 173.99 0) (unit 1)
     (in_bom yes) (on_board yes) (fields_autoplaced)
@@
     (pin "NO")
   )
+  (symbol (lib_id "Mechanical:MountingHole") (at 264.16 146.05 0) (unit 1)
+    (in_bom yes) (on_board yes) (fields_autoplaced)
+    (property "Reference" "H7" (id 0) (at 266.7 144.7799 0)
+      (effects (font (size 1.27 1.27)) (justify left))
+    )
+    (property "Value" "MountingHole" (id 1) (at 266.7 147.3199 0)
+      (effects (font (size 1.27 1.27)) (justify left))
+    )
+    (property "Footprint" "MountingHole:MountingHole_3.2mm_M3" (id 2) (at 264.16 146.05 0)
+      (effects (font (size 1.27 1.27)) hide)
+    )
+    (property "Datasheet" "~" (id 3) (at 264.16 146.05 0)
+      (effects (font (size 1.27 1.27)) hide)
+    )
+  )
   (symbol (lib_id "Connector_Generic:Conn_01x02") (at 74.93 186.69 270) (unit 1)
     (in_bom yes) (on_board yes) (fields_autoplaced)
@@
     (pin "1")
     (pin "2")
+  )
+  (symbol (lib_id "Mechanical:MountingHole") (at 241.3 156.21 0) (unit 1)
+    (in_bom yes) (on_board yes) (fields_autoplaced)
+    (property "Reference" "H6" (id 0) (at 243.84 154.9399 0)
+      (effects (font (size 1.27 1.27)) (justify left))
+    )
+    (property "Value" "MountingHole" (id 1) (at 243.84 157.4799 0)
+      (effects (font (size 1.27 1.27)) (justify left))
+    )
+    (property "Footprint" "MountingHole:MountingHole_3.2mm_M3" (id 2) (at 241.3 156.21 0)
+      (effects (font (size 1.27 1.27)) hide)
+    )
+    (property "Datasheet" "~" (id 3) (at 241.3 156.21 0)
+      (effects (font (size 1.27 1.27)) hide)
+    )
   )
   (symbol (lib_id "Device:R") (at 185.42 58.42 90) (unit 1)
@@
     (pin "2")
   )
-  (symbol (lib_id "Mechanical:MountingHole") (at 153.67 186.69 0) (unit 1)
-    (in_bom yes) (on_board yes) (fields_autoplaced)
-    (property "Reference" "H4" (id 0) (at 156.21 185.4199 0)
-      (effects (font (size 1.27 1.27)) (justify left))
-    )
-    (property "Value" "MountingHole" (id 1) (at 156.21 187.9599 0)
-      (effects (font (size 1.27 1.27)) (justify left))
-    )
-    (property "Footprint" "MountingHole:MountingHole_3.2mm_M3" (id 2) (at 153.67 186.69 0)
-      (effects (font (size 1.27 1.27)) hide)
-    )
-    (property "Datasheet" "~" (id 3) (at 153.67 186.69 0)
+  (symbol (lib_id "Mechanical:MountingHole") (at 264.16 135.89 0) (unit 1)
+    (in_bom yes) (on_board yes) (fields_autoplaced)
+    (property "Reference" "H4" (id 0) (at 266.7 134.6199 0)
+      (effects (font (size 1.27 1.27)) (justify left))
+    )
+    (property "Value" "MountingHole" (id 1) (at 266.7 137.1599 0)
+      (effects (font (size 1.27 1.27)) (justify left))
+    )
+    (property "Footprint" "MountingHole:MountingHole_3.2mm_M3" (id 2) (at 264.16 135.89 0)
+      (effects (font (size 1.27 1.27)) hide)
+    )
+    (property "Datasheet" "~" (id 3) (at 264.16 135.89 0)
       (effects (font (size 1.27 1.27)) hide)
     )
@@
       (reference "H4") (unit 1) (value "MountingHole") (footprint "MountingHole:MountingHole_3.2mm_M3")
     )
+    (path "/995c44ee-6133-4e88-af52-eddd63b33f74"
+      (reference "H5") (unit 1) (value "MountingHole") (footprint "MountingHole:MountingHole_3.2mm_M3")
+    )
+    (path "/d8fc888e-93f1-4e52-83f5-023fbe2c750a"
+      (reference "H6") (unit 1) (value "MountingHole") (footprint "MountingHole:MountingHole_3.2mm_M3")
+    )
+    (path "/bb8a5afd-18d5-4d8d-9da8-c1eb33e6ddf9"
+      (reference "H7") (unit 1) (value "MountingHole") (footprint "MountingHole:MountingHole_3.2mm_M3")
+    )
     (path "/83c82a50-fec7-4a99-9fe0-3a09a09f005c"

Commit message: Add Rev B
Parts:
- K1, K2, K3, K4, K5: value SRD-05VDC-SL-C -> SRD-12VDC-SL-C
Connections:
- net VIN renamed 12V
Changed lines of the file:
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@@
   (title_block
     (title "Sherline CNC - Motor Board")
-    (date "2021-11-29")
-    (rev "A")
+    (date "2022-02-10")
+    (rev "B")
     (company "A.C. Wright Design")
   )
@@
     (stroke (width 0) (type default) (color 0 0 0 0))
   )
-  (global_label "VIN" (shape input) (at 83.82 102.87 90) (fields_autoplaced)
-    (effects (font (size 1.27 1.27)) (justify left))
-    (property "Intersheet References" "${INTERSHEET_REFS}" (id 0) (at 83.7406 97.4331 90)
-      (effects (font (size 1.27 1.27)) (justify left) hide)
-    )
-  )
-  (global_label "VIN" (shape input) (at 199.39 86.36 90) (fields_autoplaced)
-    (effects (font (size 1.27 1.27)) (justify left))
-    (property "Intersheet References" "${INTERSHEET_REFS}" (id 0) (at 199.3106 80.9231 90)
-      (effects (font (size 1.27 1.27)) (justify left) hide)
-    )
-  )
-  (global_label "VIN" (shape input) (at 199.39 34.29 90) (fields_autoplaced)
-    (effects (font (size 1.27 1.27)) (justify left))
-    (property "Intersheet References" "${INTERSHEET_REFS}" (id 0) (at 199.3106 28.8531 90)
-      (effects (font (size 1.27 1.27)) (justify left) hide)
-    )
-  )
-  (global_label "VIN" (shape output) (at 48.26 82.55 0) (fields_autoplaced)
-    (effects (font (size 1.27 1.27)) (justify left))
-    (property "Intersheet References" "${INTERSHEET_REFS}" (id 0) (at 53.6969 82.4706 0)
+  (global_label "12V" (shape input) (at 83.82 102.87 90) (fields_autoplaced)
+    (effects (font (size 1.27 1.27)) (justify left))
+    (property "Intersheet References" "${INTERSHEET_REFS}" (id 0) (at 83.7406 96.9493 90)
+      (effects (font (size 1.27 1.27)) (justify left) hide)
+    )
+  )
+  (global_label "12V" (shape input) (at 199.39 86.36 90) (fields_autoplaced)
+    (effects (font (size 1.27 1.27)) (justify left))
+    (property "Intersheet References" "${INTERSHEET_REFS}" (id 0) (at 199.3106 80.4393 90)
+      (effects (font (size 1.27 1.27)) (justify left) hide)
+    )
+  )
+  (global_label "12V" (shape input) (at 199.39 34.29 90) (fields_autoplaced)
+    (effects (font (size 1.27 1.27)) (justify left))
+    (property "Intersheet References" "${INTERSHEET_REFS}" (id 0) (at 199.3106 28.3693 90)
+      (effects (font (size 1.27 1.27)) (justify left) hide)
+    )
+  )
+  (global_label "12V" (shape output) (at 48.26 82.55 0) (fields_autoplaced)
+    (effects (font (size 1.27 1.27)) (justify left))
+    (property "Intersheet References" "${INTERSHEET_REFS}" (id 0) (at 54.1807 82.4706 0)
       (effects (font (size 1.27 1.27)) (justify left) hide)
     )
@@
     )
   )
-  (global_label "VIN" (shape input) (at 134.62 34.29 90) (fields_autoplaced)
-    (effects (font (size 1.27 1.27)) (justify left))
-    (property "Intersheet References" "${INTERSHEET_REFS}" (id 0) (at 134.5406 28.8531 90)
+  (global_label "12V" (shape input) (at 134.62 34.29 90) (fields_autoplaced)
+    (effects (font (size 1.27 1.27)) (justify left))
+    (property "Intersheet References" "${INTERSHEET_REFS}" (id 0) (at 134.5406 28.3693 90)
       (effects (font (size 1.27 1.27)) (justify left) hide)
     )
@@
     )
   )
-  (global_label "VIN" (shape input) (at 134.62 86.36 90) (fields_autoplaced)
-    (effects (font (size 1.27 1.27)) (justify left))
-    (property "Intersheet References" "${INTERSHEET_REFS}" (id 0) (at 134.5406 80.9231 90)
+  (global_label "12V" (shape input) (at 134.62 86.36 90) (fields_autoplaced)
+    (effects (font (size 1.27 1.27)) (justify left))
+    (property "Intersheet References" "${INTERSHEET_REFS}" (id 0) (at 134.5406 80.4393 90)
       (effects (font (size 1.27 1.27)) (justify left) hide)
     )
@@
     )
   )
-  (global_label "VIN" (shape input) (at 86.36 34.29 90) (fields_autoplaced)
-    (effects (font (size 1.27 1.27)) (justify left))
-    (property "Intersheet References" "${INTERSHEET_REFS}" (id 0) (at 86.2806 28.8531 90)
+  (global_label "12V" (shape input) (at 86.36 34.29 90) (fields_autoplaced)
+    (effects (font (size 1.27 1.27)) (justify left))
+    (property "Intersheet References" "${INTERSHEET_REFS}" (id 0) (at 86.2806 28.3693 90)
       (effects (font (size 1.27 1.27)) (justify left) hide)
     )
@@
     (in_bom yes) (on_board yes) (fields_autoplaced)
     (property "Reference" "K2" (id 0) (at 151.13 31.75 0))
-    (property "Value" "SRD-05VDC-SL-C" (id 1) (at 151.13 34.29 0))
+    (property "Value" "SRD-12VDC-SL-C" (id 1) (at 151.13 34.29 0))
     (property "Footprint" "SRD-05VDC-SL-C:SRD-05VDC-SL-C" (id 2) (at 151.13 41.91 0)
       (effects (font (size 1.27 1.27)) (justify left bottom) hide)
@@
     (in_bom yes) (on_board yes) (fields_autoplaced)
     (property "Reference" "K3" (id 0) (at 151.13 83.82 0))
-    (property "Value" "SRD-05VDC-SL-C" (id 1) (at 151.13 86.36 0))
+    (property "Value" "SRD-12VDC-SL-C" (id 1) (at 151.13 86.36 0))
     (property "Footprint" "SRD-05VDC-SL-C:SRD-05VDC-SL-C" (id 2) (at 151.13 93.98 0)
       (effects (font (size 1.27 1.27)) (justify left bottom) hide)
@@
     (in_bom yes) (on_board yes) (fields_autoplaced)
     (property "Reference" "K4" (id 0) (at 215.9 31.75 0))
-    (property "Value" "SRD-05VDC-SL-C" (id 1) (at 215.9 34.29 0))
+    (property "Value" "SRD-12VDC-SL-C" (id 1) (at 215.9 34.29 0))
     (property "Footprint" "SRD-05VDC-SL-C:SRD-05VDC-SL-C" (id 2) (at 215.9 41.91 0)
       (effects (font (size 1.27 1.27)) (justify left bottom) hide)
@@
     (in_bom yes) (on_board yes) (fields_autoplaced)
     (property "Reference" "K1" (id 0) (at 71.12 31.75 0))
-    (property "Value" "SRD-05VDC-SL-C" (id 1) (at 71.12 34.29 0))
+    (property "Value" "SRD-12VDC-SL-C" (id 1) (at 71.12 34.29 0))
     (property "Footprint" "SRD-05VDC-SL-C:SRD-05VDC-SL-C" (id 2) (at 71.12 41.91 0)
       (effects (font (size 1.27 1.27)) (justify left bottom) hide)
@@
     (in_bom yes) (on_board yes) (fields_autoplaced)
     (property "Reference" "K5" (id 0) (at 215.9 83.82 0))
-    (property "Value" "SRD-05VDC-SL-C" (id 1) (at 215.9 86.36 0))
+    (property "Value" "SRD-12VDC-SL-C" (id 1) (at 215.9 86.36 0))
     (property "Footprint" "SRD-05VDC-SL-C:SRD-05VDC-SL-C" (id 2) (at 215.9 93.98 0)
       (effects (font (size 1.27 1.27)) (justify left bottom) hide)
@@
     )
     (path "/ba177c26-19d0-43c4-a360-daebdb43ddd0"
-      (reference "K1") (unit 1) (value "SRD-05VDC-SL-C") (footprint "SRD-05VDC-SL-C:SRD-05VDC-SL-C")
+      (reference "K1") (unit 1) (value "SRD-12VDC-SL-C") (footprint "SRD-05VDC-SL-C:SRD-05VDC-SL-C")
     )
     (path "/1ced5472-90bf-4251-8b79-8a1090ab3400"
-      (reference "K2") (unit 1) (value "SRD-05VDC-SL-C") (footprint "SRD-05VDC-SL-C:SRD-05VDC-SL-C")
+      (reference "K2") (unit 1) (value "SRD-12VDC-SL-C") (footprint "SRD-05VDC-SL-C:SRD-05VDC-SL-C")
     )
     (path "/6feadc61-c71a-4b8f-8cda-f061fe372ebd"
-      (reference "K3") (unit 1) (value "SRD-05VDC-SL-C") (footprint "SRD-05VDC-SL-C:SRD-05VDC-SL-C")
+      (reference "K3") (unit 1) (value "SRD-12VDC-SL-C") (footprint "SRD-05VDC-SL-C:SRD-05VDC-SL-C")
     )
     (path "/94932266-8186-4c4f-afb4-5c719d755afb"
-      (reference "K4") (unit 1) (value "SRD-05VDC-SL-C") (footprint "SRD-05VDC-SL-C:SRD-05VDC-SL-C")
+      (reference "K4") (unit 1) (value "SRD-12VDC-SL-C") (footprint "SRD-05VDC-SL-C:SRD-05VDC-SL-C")
     )
     (path "/c8f7257d-41db-47c0-96c3-95927e5035ac"
-      (reference "K5") (unit 1) (value "SRD-05VDC-SL-C") (footprint "SRD-05VDC-SL-C:SRD-05VDC-SL-C")
+      (reference "K5") (unit 1) (value "SRD-12VDC-SL-C") (footprint "SRD-05VDC-SL-C:SRD-05VDC-SL-C")
     )
     (path "/ff42c4c4-1b4f-47db-aa04-7753bc2b86ba"
